File: iCE40HX1K-EVB_Rev_B.kicad_pcb (KiCad board)
At the start: 4 copper layers, 50 x 50 mm, 85 parts, among them U1 W25Q16BVSSIG(SOIC-8_208mil), U2 SY8009AAAC(SOT23-5), U3 SY8009AAAC(SOT23-5), U4 ICE40HX1K-VQ100(VQFP100), U5 K6R4016V1D-TC10(TSOP-44)

Commit message: regymm modified version
Parts:
- added J1: PMOD1, Connector_PinHeader_2.54mm:PinHeader_2x06_P2.54mm_Vertical, F.Cu at (161.0, 50.8)
- added J2: PMOD1, Connector_PinHeader_2.54mm:PinHeader_2x06_P2.54mm_Vertical, F.Cu at (161.0, 27.9)
- added J3: UART, Connector_PinHeader_2.54mm:PinHeader_1x10_P2.54mm_Vertical, F.Cu at (143.3, 58.4)
- added J4: PROG, Connector_PinHeader_2.54mm:PinHeader_1x10_P2.54mm_Vertical, F.Cu at (117.9, 58.4)
- added J5: 1V2, Connector_PinHeader_2.54mm:PinHeader_1x01_P2.54mm_Vertical, F.Cu at (156.0, 27.9)
- CR1: footprint OLIMEX_Crystal-FP:Oscillator_7.0x5.0mm -> Crystal:Crystal_SMD_3225-4Pin_3.2x2.5mm_HandSoldering
Connections:
- net Net-(PGM1-Pad3) renamed /FT_RxD
- net Net-(PGM1-Pad4) renamed /FT_TxD
Routing:
- net +3V3: track 114.4 -> 199.6 mm
- net +1V2: track 97.0 -> 181.5 mm
- net /iCE40-SDO: track 37.8 -> 116.9 mm
- net GND: track 306.1 -> 384.1 mm
- net /iCE40-SCK: track 32.8 -> 105.6 mm
- net /FT_RxD: track 19.5 -> 79.2 mm, vias 1 -> 2
- net /iCE40-SDI: track 40.5 -> 98.3 mm
- net /iCE40-SS_B: track 45.8 -> 100.2 mm
- net /FT_TxD: track 24.4 -> 77.5 mm, vias 1 -> 2
- net /SA5: track 36.7 -> 89.6 mm
- net /SD7: track 22.7 -> 72.3 mm
- net /SRAM_#WE: track 17.3 -> 65.4 mm
- net /SD5: track 24.1 -> 70.6 mm
- net /SD6: track 24.0 -> 68.9 mm
- net /SD3: track 24.0 -> 66.6 mm
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Other:
- board size 50 x 50 mm -> 50.1 x 95.7 mm
- board text added: "%regymm"
