File: iCE40HX1K-EVB_Rev_B.sch (KiCad schematic (older format))
At the start: 72 parts, among them U1 W25Q16BVSSIG(SOIC-8_208mil), U2 SY8009AAAC(SOT23-5), U3 SY8009AAAC(SOT23-5), U4 ICE40HX1K-VQ100(VQFP100), U5 K6R4016V1D-TC10(TSOP-44)

Commit message: regymm modified version
Parts:
- added J1, J2: PMOD1, Connector_PinHeader_2.54mm:PinHeader_2x06_P2.54mm_Vertical, symbol Connector_Generic:Conn_02x06_Odd_Even
- added J3: UART, Connector_PinHeader_2.54mm:PinHeader_1x10_P2.54mm_Vertical, symbol Connector:Conn_01x10_Male
- added J4: PROG, Connector_PinHeader_2.54mm:PinHeader_1x10_P2.54mm_Vertical, symbol Connector:Conn_01x10_Male
- added J5: 1V2, Connector_PinHeader_2.54mm:PinHeader_1x01_P2.54mm_Vertical, symbol Connector:Conn_01x01_Male
- 3.3V_E1, RxD_E1, TxD_E1: symbol SJ -> iCE40HX1K-EVB_Rev_B-rescue:SJ-iCE40HX1K-EVB_Rev_B-rescue
- BUT1, BUT2, RESET1: symbol T1107A(6x3,8x2,5MM) -> iCE40HX1K-EVB_Rev_B-rescue:T1107A(6x3,8x2,5MM)-iCE40HX1K-EVB_Rev_B-rescue
- C1, C10, C11, C12, C13, C14, C15, C16, C17, C18, C19, C2, C20, C21, C22, C23, C24, C25, C26, C27, C28, C3, C4, C5, C6, C7, C8, C9: symbol C -> iCE40HX1K-EVB_Rev_B-rescue:C-iCE40HX1K-EVB_Rev_B-rescue
- CDone1, LED1, LED2, PWRLED1: symbol LED -> iCE40HX1K-EVB_Rev_B-rescue:LED-iCE40HX1K-EVB_Rev_B-rescue
- CR1: footprint OLIMEX_Crystal-FP:Oscillator_7.0x5.0mm -> Crystal:Crystal_SMD_3225-4Pin_3.2x2.5mm_HandSoldering; symbol Oscillator-100MHZ_TXC-7W -> iCE40HX1K-EVB_Rev_B-rescue:Oscillator-100MHZ_TXC-7W-iCE40HX1K-EVB_Rev_B-rescue
- D1: symbol SMBJ6.0A -> iCE40HX1K-EVB_Rev_B-rescue:SMBJ6.0A-iCE40HX1K-EVB_Rev_B-rescue
- D2: symbol D_Schottky -> iCE40HX1K-EVB_Rev_B-rescue:D_Schottky-iCE40HX1K-EVB_Rev_B-rescue
- FUSE1: symbol FSMD035 -> iCE40HX1K-EVB_Rev_B-rescue:FSMD035-iCE40HX1K-EVB_Rev_B-rescue
- GND1: symbol TESTPAD -> iCE40HX1K-EVB_Rev_B-rescue:TESTPAD-iCE40HX1K-EVB_Rev_B-rescue
- GPIO1: symbol BH34S -> iCE40HX1K-EVB_Rev_B-rescue:BH34S-iCE40HX1K-EVB_Rev_B-rescue
- L1, L2: symbol L -> iCE40HX1K-EVB_Rev_B-rescue:L-iCE40HX1K-EVB_Rev_B-rescue
- PGM1: symbol BH10S -> iCE40HX1K-EVB_Rev_B-rescue:BH10S-iCE40HX1K-EVB_Rev_B-rescue
- PWR1: symbol PWR-JAKPWR_JACK_UNI_MILLING -> iCE40HX1K-EVB_Rev_B-rescue:PWR-JAKPWR_JACK_UNI_MILLING-iCE40HX1K-EVB_Rev_B-rescue
- R1, R10, R11, R12, R13, R14, R15, R16, R17, R18, R19, R2, R3, R4, R5, R6, R7, R8, R9: symbol R -> iCE40HX1K-EVB_Rev_B-rescue:R-iCE40HX1K-EVB_Rev_B-rescue
- U1: symbol W25Q16BV -> iCE40HX1K-EVB_Rev_B-rescue:W25Q16BV-iCE40HX1K-EVB_Rev_B-rescue
- U2, U3: symbol SY8009AAAC(SOT23-5) -> iCE40HX1K-EVB_Rev_B-rescue:SY8009AAAC(SOT23-5)-iCE40HX1K-EVB_Rev_B-rescue
- U4: symbol ICE40HX1K-VQ100(VQFP100) -> iCE40HX1K-EVB_Rev_B-rescue:ICE40HX1K-VQ100(VQFP100)-iCE40HX1K-EVB_Rev_B-rescue
- U5: symbol K6R4016V1D-TC10(TSOP-44) -> iCE40HX1K-EVB_Rev_B-rescue:K6R4016V1D-TC10(TSOP-44)-iCE40HX1K-EVB_Rev_B-rescue
Connections:
- net labels added: FT_RxD, FT_TxD
- wire segments 374 -> 497
